Commit message: v1.7

File: simulation/models/ur5/ur5.urdf (robot description, URDF)
Before this commit: robot ur5_robot, 11 links, 10 joints
Links:
- link base_link_inertia: geometry collision mesh filename=ur_description/meshes/ur5/collision/base.stl; visual mesh filename=ur_description/meshes/ur5/visual/base.dae
- link forearm_link: geometry collision mesh filename=ur_description/meshes/ur5/collision/forearm.stl; visual mesh filename=ur_description/meshes/ur5/visual/forearm.dae
- link shoulder_link: geometry collision mesh filename=ur_description/meshes/ur5/collision/shoulder.stl; visual mesh filename=ur_description/meshes/ur5/visual/shoulder.dae
- link upper_arm_link: geometry collision mesh filename=ur_description/meshes/ur5/collision/upperarm.stl; visual mesh filename=ur_description/meshes/ur5/visual/upperarm.dae
- link wrist_1_link: geometry collision mesh filename=ur_description/meshes/ur5/collision/wrist1.stl; visual mesh filename=ur_description/meshes/ur5/visual/wrist1.dae
- link wrist_2_link: geometry collision mesh filename=ur_description/meshes/ur5/collision/wrist2.stl; visual mesh filename=ur_description/meshes/ur5/visual/wrist2.dae
- link wrist_3_link: geometry collision mesh filename=ur_description/meshes/ur5/collision/wrist3.stl; visual mesh filename=ur_description/meshes/ur5/visual/wrist3.dae

File: simulation/models/ur5/ur_description/urdf/inc/ur10_macro.xacro (robot description, xacro)
@@ -19,8 +19,8 @@
   <xacro:macro name="ur10_robot" params="
    prefix
-   joint_limits_parameters_file:='/home/shijie/robot/simulation/models/ur5/ur_description/config/ur10/joint_limits.yaml'
-   kinematics_parameters_file:='/home/shijie/robot/simulation/models/ur5/ur_description/config/ur10/default_kinematics.yaml'
-   physical_parameters_file:='/home/shijie/robot/simulation/models/ur5/ur_description/config/ur10/physical_parameters.yaml'
-   visual_parameters_file:='/home/shijie/robot/simulation/models/ur5/ur_description/config/ur10/visual_parameters.yaml'
+   joint_limits_parameters_file:='$(find ur_description)/config/ur10/joint_limits.yaml'
+   kinematics_parameters_file:='$(find ur_description)/config/ur10/default_kinematics.yaml'
+   physical_parameters_file:='$(find ur_description)/config/ur10/physical_parameters.yaml'
+   visual_parameters_file:='$(find ur_description)/config/ur10/visual_parameters.yaml'
    transmission_hw_interface:=hardware_interface/PositionJointInterface
    safety_limits:=false
@@ -28,5 +28,5 @@
    safety_k_position:=20"
   >
-    <xacro:include filename="/home/shijie/robot/simulation/models/ur5/ur_description/urdf/inc/ur_macro.xacro"/>
+    <xacro:include filename="$(find ur_description)/urdf/inc/ur_macro.xacro"/>
     <xacro:ur_robot
       prefix="${prefix}"

File: simulation/models/ur5/ur_description/urdf/inc/ur10e_macro.xacro (robot description, xacro)
@@ -19,8 +19,8 @@
   <xacro:macro name="ur10e_robot" params="
    prefix
-   joint_limits_parameters_file:='/home/shijie/robot/simulation/models/ur5/ur_description/config/ur10e/joint_limits.yaml'
-   kinematics_parameters_file:='/home/shijie/robot/simulation/models/ur5/ur_description/config/ur10e/default_kinematics.yaml'
-   physical_parameters_file:='/home/shijie/robot/simulation/models/ur5/ur_description/config/ur10e/physical_parameters.yaml'
-   visual_parameters_file:='/home/shijie/robot/simulation/models/ur5/ur_description/config/ur10e/visual_parameters.yaml'
+   joint_limits_parameters_file:='$(find ur_description)/config/ur10e/joint_limits.yaml'
+   kinematics_parameters_file:='$(find ur_description)/config/ur10e/default_kinematics.yaml'
+   physical_parameters_file:='$(find ur_description)/config/ur10e/physical_parameters.yaml'
+   visual_parameters_file:='$(find ur_description)/config/ur10e/visual_parameters.yaml'
    transmission_hw_interface:=hardware_interface/PositionJointInterface
    safety_limits:=false
@@ -28,5 +28,5 @@
    safety_k_position:=20"
   >
-    <xacro:include filename="/home/shijie/robot/simulation/models/ur5/ur_description/urdf/inc/ur_macro.xacro"/>
+    <xacro:include filename="$(find ur_description)/urdf/inc/ur_macro.xacro"/>
     <xacro:ur_robot
       prefix="${prefix}"

File: simulation/models/ur5/ur_description/urdf/inc/ur12e_macro.xacro (robot description, xacro)
@@ -19,8 +19,8 @@
   <xacro:macro name="ur12e_robot" params="
    prefix
-   joint_limits_parameters_file:='/home/shijie/robot/simulation/models/ur5/ur_description/config/ur12e/joint_limits.yaml'
-   kinematics_parameters_file:='/home/shijie/robot/simulation/models/ur5/ur_description/config/ur12e/default_kinematics.yaml'
-   physical_parameters_file:='/home/shijie/robot/simulation/models/ur5/ur_description/config/ur12e/physical_parameters.yaml'
-   visual_parameters_file:='/home/shijie/robot/simulation/models/ur5/ur_description/config/ur12e/visual_parameters.yaml'
+   joint_limits_parameters_file:='$(find ur_description)/config/ur12e/joint_limits.yaml'
+   kinematics_parameters_file:='$(find ur_description)/config/ur12e/default_kinematics.yaml'
+   physical_parameters_file:='$(find ur_description)/config/ur12e/physical_parameters.yaml'
+   visual_parameters_file:='$(find ur_description)/config/ur12e/visual_parameters.yaml'
    transmission_hw_interface:=hardware_interface/PositionJointInterface
    safety_limits:=false
@@ -28,5 +28,5 @@
    safety_k_position:=20"
   >
-    <xacro:include filename="/home/shijie/robot/simulation/models/ur5/ur_description/urdf/inc/ur_macro.xacro"/>
+    <xacro:include filename="$(find ur_description)/urdf/inc/ur_macro.xacro"/>
     <xacro:ur_robot
       prefix="${prefix}"

File: simulation/models/ur5/ur_description/urdf/inc/ur15_macro.xacro (robot description, xacro)
@@ -19,8 +19,8 @@
   <xacro:macro name="ur15_robot" params="
    prefix
-   joint_limits_parameters_file:='/home/shijie/robot/simulation/models/ur5/ur_description/config/ur15/joint_limits.yaml'
-   kinematics_parameters_file:='/home/shijie/robot/simulation/models/ur5/ur_description/config/ur15/default_kinematics.yaml'
-   physical_parameters_file:='/home/shijie/robot/simulation/models/ur5/ur_description/config/ur15/physical_parameters.yaml'
-   visual_parameters_file:='/home/shijie/robot/simulation/models/ur5/ur_description/config/ur15/visual_parameters.yaml'
+   joint_limits_parameters_file:='$(find ur_description)/config/ur15/joint_limits.yaml'
+   kinematics_parameters_file:='$(find ur_description)/config/ur15/default_kinematics.yaml'
+   physical_parameters_file:='$(find ur_description)/config/ur15/physical_parameters.yaml'
+   visual_parameters_file:='$(find ur_description)/config/ur15/visual_parameters.yaml'
    transmission_hw_interface:=hardware_interface/PositionJointInterface
    safety_limits:=false
@@ -28,5 +28,5 @@
    safety_k_position:=20"
   >
-    <xacro:include filename="/home/shijie/robot/simulation/models/ur5/ur_description/urdf/inc/ur_macro.xacro"/>
+    <xacro:include filename="$(find ur_description)/urdf/inc/ur_macro.xacro"/>
     <xacro:ur_robot
       prefix="${prefix}"

File: simulation/models/ur5/ur_description/urdf/inc/ur16e_macro.xacro (robot description, xacro)
@@ -19,8 +19,8 @@
   <xacro:macro name="ur16e_robot" params="
    prefix
-   joint_limits_parameters_file:='/home/shijie/robot/simulation/models/ur5/ur_description/config/ur16e/joint_limits.yaml'
-   kinematics_parameters_file:='/home/shijie/robot/simulation/models/ur5/ur_description/config/ur16e/default_kinematics.yaml'
-   physical_parameters_file:='/home/shijie/robot/simulation/models/ur5/ur_description/config/ur16e/physical_parameters.yaml'
-   visual_parameters_file:='/home/shijie/robot/simulation/models/ur5/ur_description/config/ur16e/visual_parameters.yaml'
+   joint_limits_parameters_file:='$(find ur_description)/config/ur16e/joint_limits.yaml'
+   kinematics_parameters_file:='$(find ur_description)/config/ur16e/default_kinematics.yaml'
+   physical_parameters_file:='$(find ur_description)/config/ur16e/physical_parameters.yaml'
+   visual_parameters_file:='$(find ur_description)/config/ur16e/visual_parameters.yaml'
    transmission_hw_interface:=hardware_interface/PositionJointInterface
    safety_limits:=false
@@ -28,5 +28,5 @@
    safety_k_position:=20"
   >
-    <xacro:include filename="/home/shijie/robot/simulation/models/ur5/ur_description/urdf/inc/ur_macro.xacro"/>
+    <xacro:include filename="$(find ur_description)/urdf/inc/ur_macro.xacro"/>
     <xacro:ur_robot
       prefix="${prefix}"

File: simulation/models/ur5/ur_description/urdf/inc/ur18_macro.xacro (robot description, xacro)
@@ -19,8 +19,8 @@
   <xacro:macro name="ur18_robot" params="
    prefix
-   joint_limits_parameters_file:='/home/shijie/robot/simulation/models/ur5/ur_description/config/ur18/joint_limits.yaml'
-   kinematics_parameters_file:='/home/shijie/robot/simulation/models/ur5/ur_description/config/ur18/default_kinematics.yaml'
-   physical_parameters_file:='/home/shijie/robot/simulation/models/ur5/ur_description/config/ur18/physical_parameters.yaml'
-   visual_parameters_file:='/home/shijie/robot/simulation/models/ur5/ur_description/config/ur18/visual_parameters.yaml'
+   joint_limits_parameters_file:='$(find ur_description)/config/ur18/joint_limits.yaml'
+   kinematics_parameters_file:='$(find ur_description)/config/ur18/default_kinematics.yaml'
+   physical_parameters_file:='$(find ur_description)/config/ur18/physical_parameters.yaml'
+   visual_parameters_file:='$(find ur_description)/config/ur18/visual_parameters.yaml'
    transmission_hw_interface:=hardware_interface/PositionJointInterface
    safety_limits:=false
@@ -28,5 +28,5 @@
    safety_k_position:=20"
   >
-    <xacro:include filename="/home/shijie/robot/simulation/models/ur5/ur_description/urdf/inc/ur_macro.xacro"/>
+    <xacro:include filename="$(find ur_description)/urdf/inc/ur_macro.xacro"/>
     <xacro:ur_robot
       prefix="${prefix}"

File: simulation/models/ur5/ur_description/urdf/inc/ur20_macro.xacro (robot description, xacro)
@@ -19,8 +19,8 @@
   <xacro:macro name="ur20_robot" params="
    prefix
-   joint_limits_parameters_file:='/home/shijie/robot/simulation/models/ur5/ur_description/config/ur20/joint_limits.yaml'
-   kinematics_parameters_file:='/home/shijie/robot/simulation/models/ur5/ur_description/config/ur20/default_kinematics.yaml'
-   physical_parameters_file:='/home/shijie/robot/simulation/models/ur5/ur_description/config/ur20/physical_parameters.yaml'
-   visual_parameters_file:='/home/shijie/robot/simulation/models/ur5/ur_description/config/ur20/visual_parameters.yaml'
+   joint_limits_parameters_file:='$(find ur_description)/config/ur20/joint_limits.yaml'
+   kinematics_parameters_file:='$(find ur_description)/config/ur20/default_kinematics.yaml'
+   physical_parameters_file:='$(find ur_description)/config/ur20/physical_parameters.yaml'
+   visual_parameters_file:='$(find ur_description)/config/ur20/visual_parameters.yaml'
    transmission_hw_interface:=hardware_interface/PositionJointInterface
    safety_limits:=false
@@ -28,5 +28,5 @@
    safety_k_position:=20"
   >
-    <xacro:include filename="/home/shijie/robot/simulation/models/ur5/ur_description/urdf/inc/ur_macro.xacro"/>
+    <xacro:include filename="$(find ur_description)/urdf/inc/ur_macro.xacro"/>
     <xacro:ur_robot
       prefix="${prefix}"

File: simulation/models/ur5/ur_description/urdf/inc/ur30_macro.xacro (robot description, xacro)
@@ -19,8 +19,8 @@
   <xacro:macro name="ur30_robot" params="
    prefix
-   joint_limits_parameters_file:='/home/shijie/robot/simulation/models/ur5/ur_description/config/ur30/joint_limits.yaml'
-   kinematics_parameters_file:='/home/shijie/robot/simulation/models/ur5/ur_description/config/ur30/default_kinematics.yaml'
-   physical_parameters_file:='/home/shijie/robot/simulation/models/ur5/ur_description/config/ur30/physical_parameters.yaml'
-   visual_parameters_file:='/home/shijie/robot/simulation/models/ur5/ur_description/config/ur30/visual_parameters.yaml'
+   joint_limits_parameters_file:='$(find ur_description)/config/ur30/joint_limits.yaml'
+   kinematics_parameters_file:='$(find ur_description)/config/ur30/default_kinematics.yaml'
+   physical_parameters_file:='$(find ur_description)/config/ur30/physical_parameters.yaml'
+   visual_parameters_file:='$(find ur_description)/config/ur30/visual_parameters.yaml'
    transmission_hw_interface:=hardware_interface/PositionJointInterface
    safety_limits:=false
@@ -28,5 +28,5 @@
    safety_k_position:=20"
   >
-    <xacro:include filename="/home/shijie/robot/simulation/models/ur5/ur_description/urdf/inc/ur_macro.xacro"/>
+    <xacro:include filename="$(find ur_description)/urdf/inc/ur_macro.xacro"/>
     <xacro:ur_robot
       prefix="${prefix}"

File: simulation/models/ur5/ur_description/urdf/inc/ur3_macro.xacro (robot description, xacro)
@@ -19,8 +19,8 @@
   <xacro:macro name="ur3_robot" params="
    prefix
-   joint_limits_parameters_file:='/home/shijie/robot/simulation/models/ur5/ur_description/config/ur3/joint_limits.yaml'
-   kinematics_parameters_file:='/home/shijie/robot/simulation/models/ur5/ur_description/config/ur3/default_kinematics.yaml'
-   physical_parameters_file:='/home/shijie/robot/simulation/models/ur5/ur_description/config/ur3/physical_parameters.yaml'
-   visual_parameters_file:='/home/shijie/robot/simulation/models/ur5/ur_description/config/ur3/visual_parameters.yaml'
+   joint_limits_parameters_file:='$(find ur_description)/config/ur3/joint_limits.yaml'
+   kinematics_parameters_file:='$(find ur_description)/config/ur3/default_kinematics.yaml'
+   physical_parameters_file:='$(find ur_description)/config/ur3/physical_parameters.yaml'
+   visual_parameters_file:='$(find ur_description)/config/ur3/visual_parameters.yaml'
    transmission_hw_interface:=hardware_interface/PositionJointInterface
    safety_limits:=false
@@ -28,5 +28,5 @@
    safety_k_position:=20"
   >
-    <xacro:include filename="/home/shijie/robot/simulation/models/ur5/ur_description/urdf/inc/ur_macro.xacro"/>
+    <xacro:include filename="$(find ur_description)/urdf/inc/ur_macro.xacro"/>
     <xacro:ur_robot
       prefix="${prefix}"

File: simulation/models/ur5/ur_description/urdf/inc/ur3e_macro.xacro (robot description, xacro)
@@ -19,8 +19,8 @@
   <xacro:macro name="ur3e_robot" params="
    prefix
-   joint_limits_parameters_file:='/home/shijie/robot/simulation/models/ur5/ur_description/config/ur3e/joint_limits.yaml'
-   kinematics_parameters_file:='/home/shijie/robot/simulation/models/ur5/ur_description/config/ur3e/default_kinematics.yaml'
-   physical_parameters_file:='/home/shijie/robot/simulation/models/ur5/ur_description/config/ur3e/physical_parameters.yaml'
-   visual_parameters_file:='/home/shijie/robot/simulation/models/ur5/ur_description/config/ur3e/visual_parameters.yaml'
+   joint_limits_parameters_file:='$(find ur_description)/config/ur3e/joint_limits.yaml'
+   kinematics_parameters_file:='$(find ur_description)/config/ur3e/default_kinematics.yaml'
+   physical_parameters_file:='$(find ur_description)/config/ur3e/physical_parameters.yaml'
+   visual_parameters_file:='$(find ur_description)/config/ur3e/visual_parameters.yaml'
    transmission_hw_interface:=hardware_interface/PositionJointInterface
    safety_limits:=false
@@ -28,5 +28,5 @@
    safety_k_position:=20"
   >
-    <xacro:include filename="/home/shijie/robot/simulation/models/ur5/ur_description/urdf/inc/ur_macro.xacro"/>
+    <xacro:include filename="$(find ur_description)/urdf/inc/ur_macro.xacro"/>
     <xacro:ur_robot
       prefix="${prefix}"

File: simulation/models/ur5/ur_description/urdf/inc/ur5_macro.xacro (robot description, xacro)
@@ -19,8 +19,8 @@
   <xacro:macro name="ur5_robot" params="
    prefix
-   joint_limits_parameters_file:='/home/shijie/robot/simulation/models/ur5/ur_description/config/ur5/joint_limits.yaml'
-   kinematics_parameters_file:='/home/shijie/robot/simulation/models/ur5/ur_description/config/ur5/default_kinematics.yaml'
-   physical_parameters_file:='/home/shijie/robot/simulation/models/ur5/ur_description/config/ur5/physical_parameters.yaml'
-   visual_parameters_file:='/home/shijie/robot/simulation/models/ur5/ur_description/config/ur5/visual_parameters.yaml'
+   joint_limits_parameters_file:='$(find ur_description)/config/ur5/joint_limits.yaml'
+   kinematics_parameters_file:='$(find ur_description)/config/ur5/default_kinematics.yaml'
+   physical_parameters_file:='$(find ur_description)/config/ur5/physical_parameters.yaml'
+   visual_parameters_file:='$(find ur_description)/config/ur5/visual_parameters.yaml'
    transmission_hw_interface:=hardware_interface/PositionJointInterface
    safety_limits:=false
@@ -28,5 +28,5 @@
    safety_k_position:=20"
   >
-    <xacro:include filename="/home/shijie/robot/simulation/models/ur5/ur_description/urdf/inc/ur_macro.xacro"/>
+    <xacro:include filename="$(find ur_description)/urdf/inc/ur_macro.xacro"/>
     <xacro:ur_robot
       prefix="${prefix}"

File: simulation/models/ur5/ur_description/urdf/inc/ur5e_macro.xacro (robot description, xacro)
@@ -19,8 +19,8 @@
   <xacro:macro name="ur5e_robot" params="
    prefix
-   joint_limits_parameters_file:='/home/shijie/robot/simulation/models/ur5/ur_description/config/ur5e/joint_limits.yaml'
-   kinematics_parameters_file:='/home/shijie/robot/simulation/models/ur5/ur_description/config/ur5e/default_kinematics.yaml'
-   physical_parameters_file:='/home/shijie/robot/simulation/models/ur5/ur_description/config/ur5e/physical_parameters.yaml'
-   visual_parameters_file:='/home/shijie/robot/simulation/models/ur5/ur_description/config/ur5e/visual_parameters.yaml'
+   joint_limits_parameters_file:='$(find ur_description)/config/ur5e/joint_limits.yaml'
+   kinematics_parameters_file:='$(find ur_description)/config/ur5e/default_kinematics.yaml'
+   physical_parameters_file:='$(find ur_description)/config/ur5e/physical_parameters.yaml'
+   visual_parameters_file:='$(find ur_description)/config/ur5e/visual_parameters.yaml'
    transmission_hw_interface:=hardware_interface/PositionJointInterface
    safety_limits:=false
@@ -28,5 +28,5 @@
    safety_k_position:=20"
   >
-    <xacro:include filename="/home/shijie/robot/simulation/models/ur5/ur_description/urdf/inc/ur_macro.xacro"/>
+    <xacro:include filename="$(find ur_description)/urdf/inc/ur_macro.xacro"/>
     <xacro:ur_robot
       prefix="${prefix}"

File: simulation/models/ur5/ur_description/urdf/inc/ur7e_macro.xacro (robot description, xacro)
@@ -19,8 +19,8 @@
   <xacro:macro name="ur7e_robot" params="
    prefix
-   joint_limits_parameters_file:='/home/shijie/robot/simulation/models/ur5/ur_description/config/ur7e/joint_limits.yaml'
-   kinematics_parameters_file:='/home/shijie/robot/simulation/models/ur5/ur_description/config/ur7e/default_kinematics.yaml'
-   physical_parameters_file:='/home/shijie/robot/simulation/models/ur5/ur_description/config/ur7e/physical_parameters.yaml'
-   visual_parameters_file:='/home/shijie/robot/simulation/models/ur5/ur_description/config/ur7e/visual_parameters.yaml'
+   joint_limits_parameters_file:='$(find ur_description)/config/ur7e/joint_limits.yaml'
+   kinematics_parameters_file:='$(find ur_description)/config/ur7e/default_kinematics.yaml'
+   physical_parameters_file:='$(find ur_description)/config/ur7e/physical_parameters.yaml'
+   visual_parameters_file:='$(find ur_description)/config/ur7e/visual_parameters.yaml'
    transmission_hw_interface:=hardware_interface/PositionJointInterface
    safety_limits:=false
@@ -28,5 +28,5 @@
    safety_k_position:=20"
   >
-    <xacro:include filename="/home/shijie/robot/simulation/models/ur5/ur_description/urdf/inc/ur_macro.xacro"/>
+    <xacro:include filename="$(find ur_description)/urdf/inc/ur_macro.xacro"/>
     <xacro:ur_robot
       prefix="${prefix}"

File: simulation/models/ur5/ur_description/urdf/inc/ur8long_macro.xacro (robot description, xacro)
@@ -19,8 +19,8 @@
   <xacro:macro name="ur8long_robot" params="
    prefix
-   joint_limits_parameters_file:='/home/shijie/robot/simulation/models/ur5/ur_description/config/ur8long/joint_limits.yaml'
-   kinematics_parameters_file:='/home/shijie/robot/simulation/models/ur5/ur_description/config/ur8long/default_kinematics.yaml'
-   physical_parameters_file:='/home/shijie/robot/simulation/models/ur5/ur_description/config/ur8long/physical_parameters.yaml'
-   visual_parameters_file:='/home/shijie/robot/simulation/models/ur5/ur_description/config/ur8long/visual_parameters.yaml'
+   joint_limits_parameters_file:='$(find ur_description)/config/ur8long/joint_limits.yaml'
+   kinematics_parameters_file:='$(find ur_description)/config/ur8long/default_kinematics.yaml'
+   physical_parameters_file:='$(find ur_description)/config/ur8long/physical_parameters.yaml'
+   visual_parameters_file:='$(find ur_description)/config/ur8long/visual_parameters.yaml'
    transmission_hw_interface:=hardware_interface/PositionJointInterface
    safety_limits:=false
@@ -28,5 +28,5 @@
    safety_k_position:=20"
   >
-    <xacro:include filename="/home/shijie/robot/simulation/models/ur5/ur_description/urdf/inc/ur_macro.xacro"/>
+    <xacro:include filename="$(find ur_description)/urdf/inc/ur_macro.xacro"/>
     <xacro:ur_robot
       prefix="${prefix}"

File: simulation/models/ur5/ur_description/urdf/inc/ur_macro.xacro (robot description, xacro)
@@ -42,6 +42,6 @@
      - Muhammad Asif Rana
   -->
-  <xacro:include filename="/home/shijie/robot/simulation/models/ur5/ur_description/urdf/inc/ur_transmissions.xacro" />
-  <xacro:include filename="/home/shijie/robot/simulation/models/ur5/ur_description/urdf/inc/ur_common.xacro" />
+  <xacro:include filename="$(find ur_description)/urdf/inc/ur_transmissions.xacro" />
+  <xacro:include filename="$(find ur_description)/urdf/inc/ur_common.xacro" />
   <xacro:macro name="ur_robot" params="
     prefix

File: simulation/models/ur5/ur_description/urdf/ur.xacro (robot description, xacro)
@@ -2,5 +2,5 @@
 <robot xmlns:xacro="http://wiki.ros.org/xacro" name="$(arg robot_model)_robot">
    <!-- import main macro -->
-   <xacro:include filename="/home/shijie/robot/simulation/models/ur5/ur_description/urdf/inc/ur_macro.xacro"/>
+   <xacro:include filename="$(find ur_description)/urdf/inc/ur_macro.xacro"/>
    <!-- parameters -->
    <xacro:arg name="joint_limit_params" default=""/>

File: simulation/models/ur5/ur_description/urdf/ur10.xacro (robot description, xacro)
@@ -14,5 +14,5 @@
     Refer to 'inc/ur_macro.xacro' for more information.
   -->
-  <xacro:include filename="/home/shijie/robot/simulation/models/ur5/ur_description/urdf/inc/ur10_macro.xacro"/>
+  <xacro:include filename="$(find ur_description)/urdf/inc/ur10_macro.xacro"/>
   <xacro:ur10_robot prefix="" />
 </robot>

File: simulation/models/ur5/ur_description/urdf/ur10e.xacro (robot description, xacro)
@@ -14,5 +14,5 @@
     Refer to 'inc/ur_macro.xacro' for more information.
   -->
-  <xacro:include filename="/home/shijie/robot/simulation/models/ur5/ur_description/urdf/inc/ur10e_macro.xacro"/>
+  <xacro:include filename="$(find ur_description)/urdf/inc/ur10e_macro.xacro"/>
   <xacro:ur10e_robot prefix="" />
 </robot>
