Commit message: v1.7

File: simulation/models/ur5/ur_description/urdf/ur12e.xacro (robot description, xacro)
@@ -14,5 +14,5 @@
     Refer to 'inc/ur_macro.xacro' for more information.
   -->
-  <xacro:include filename="/home/shijie/robot/simulation/models/ur5/ur_description/urdf/inc/ur12e_macro.xacro"/>
+  <xacro:include filename="$(find ur_description)/urdf/inc/ur12e_macro.xacro"/>
   <xacro:ur12e_robot prefix="" />
 </robot>
